File: dual-pwr/dual-pwr.kicad_pcb (KiCad board)
At the start: 2 copper layers, 50 x 50 mm, 24 parts, among them J1 Screw_Terminal_01x02, J2 Screw_Terminal_01x03, J3 Conn_01x01, J4 Conn_01x01, J5 Conn_01x01, J6 Conn_01x01, Q1 2N3904, Q2 TIP122, Q3 TIP127, U1 NE5532

Commit message: dual-pwr
Parts:
- C1, C2: value 10u 35V -> 1000u 25V
- C3, C4: value 100n -> 1u 50V
- D1, D2: value D -> 2N4007
- D3: value D -> 1N5822
- R3: value 10k -> 470k
- R4: value 4k7 -> 2k2
- moved R1 1.34 mm to (90.2, 68.7)
- moved R4 1.34 mm to (85.2, 68.7)
- moved J1 1.34 mm to (54.7, 87.7)
- moved J2 1.20 mm to (75.0, 95.3)
- moved R3 0.10 mm to (94.0, 68.7)
Connections:
- net Net-(C1-Pad1) renamed +V
- net Net-(C1-Pad2) renamed GND
- net Net-(C2-Pad2) renamed -V
Routing:
- net GND: track 148.8 -> 0.00 mm
- net -V: track 133.3 -> 50.8 mm
- net +V: track 117.9 -> 56.1 mm
- net Net-(Q1-Pad3): track 34.7 -> 42.1 mm
- net Net-(Q1-Pad2): track 25.3 -> 21.6 mm
- net Net-(F1-Pad2): track 29.7 -> 28.3 mm
- net Net-(R3-Pad1): track 16.2 -> 15.0 mm
- added copper zone on B.Cu, net +V
- added copper zone on B.Cu, net -V
- added copper zone on F.Cu, net GND
Other:
- board text added: "LM358 or TL072"
