File: dual-pwr/dual-pwr.kicad_pcb (KiCad board)
At the start: 2 copper layers, 50 x 50 mm, 24 parts, among them J1 Screw_Terminal_01x02, J2 Screw_Terminal_01x03, J3 Conn_01x01, J4 Conn_01x01, J5 Conn_01x01, J6 Conn_01x01, Q1 2N3904, Q2 TIP122, Q3 TIP127, U1 NE5532

Commit message: dual-pwr
Parts:
- removed R5, R6: 10k, Resistors_ThroughHole:R_Axial_DIN0207_L6.3mm_D2.5mm_P7.62mm_Horizontal
- added RV1: 2k, Potentiometers:Potentiometer_Trimmer_Vishay_T73XW_Vertical, F.Cu at (57.2, 76.3)
- C1, C2: footprint Capacitors_ThroughHole:CP_Radial_D10.0mm_P3.50mm -> Capacitors_ThroughHole:CP_Radial_D10.0mm_P5.00mm
- C3, C4: footprint Capacitors_ThroughHole:C_Rect_L7.0mm_W4.5mm_P5.00mm -> Capacitors_ThroughHole:C_Disc_D5.0mm_W2.5mm_P5.00mm
- R2: value 10k -> 9k1
- moved F1 39.5 mm to (92.8, 81.3), turned to 90 degrees
- moved J1 39.3 mm to (75.0, 54.0), turned to 180 degrees
- moved C1 24.2 mm to (86.4, 96.6)
- moved C2 24.1 mm to (63.6, 91.5)
- moved R3 23.4 mm to (71.2, 63.6), turned to 180 degrees
- moved Q2 22.9 mm to (83.9, 53.4)
- moved Q3 22.8 mm to (61.0, 53.4)
- moved Q1 18.1 mm to (58.5, 62.3), turned to 270 degrees
- moved R2 12.8 mm to (66.7, 71.2), turned to 180 degrees
- moved D3 11.8 mm to (82.6, 81.3), turned to 180 degrees
- moved R4 10.8 mm to (78.2, 60.4), turned to 180 degrees
- moved C3 10.2 mm to (77.5, 86.4)
- moved C4 10.1 mm to (67.4, 86.4)
- moved R1 9.69 mm to (82.0, 63.6), turned to 180 degrees
- moved D2 8.55 mm to (63.6, 86.4)
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Connections:
- net Net-(Q1-Pad3) renamed VBase
- R1 pad 2: Net-(R1-Pad2) -> Vref
- R2 pad 1: Net-(R1-Pad2) -> Vref
- R2 pad 2: -V -> Net-(R2-Pad2)
- U1 pad 1: Net-(U1-Pad1) -> Net-(R3-Pad1)
- U1 pad 2: Net-(U1-Pad1) -> Vref
- U1 pad 3: Net-(R1-Pad2) -> GND
- U1 pad 5: GND -> Vref
- U1 pad 6: Net-(R1-Pad2) -> Net-(U1-Pad6)
- U1 pad 7: Net-(R3-Pad1) -> Net-(U1-Pad6)
Routing:
- net -V: track 50.8 -> 0.11 mm
- net Net-(R1-Pad2): track 42.7 -> 0.00 mm
- net +V: track 56.1 -> 14.4 mm
- net Vref: track 0.00 -> 23.7 mm
- net Net-(Q1-Pad2): track 21.6 -> 3.81 mm
- net Net-(R3-Pad1): track 15.0 -> 5.08 mm
- net Net-(R2-Pad2): track 0.00 -> 6.50 mm
- net VBase: track 42.1 -> 45.8 mm
- net Net-(F1-Pad2): track 28.3 -> 31.5 mm
- net Net-(U1-Pad6): track 0.00 -> 2.54 mm
- net Net-(U1-Pad1): track 2.54 -> 0.00 mm
- net GND: track 0.00 -> 1.65 mm
- added copper zone on F.Cu, net +V
- added copper zone on F.Cu, net -V
- added copper zone on B.Cu, net GND
- removed copper zone on B.Cu, net +V
- removed copper zone on B.Cu, net -V
- removed copper zone on F.Cu, net GND

Commit message: all
Parts:
- moved J1 22.3 mm to (96.0, 61.7), turned to 90 degrees
- moved F1 8.03 mm to (95.3, 89.0)
Routing:
- net -V: track 0.11 -> 36.0 mm
- net Net-(F1-Pad2): track 31.5 -> 20.0 mm
- net VBase: track 45.8 -> 41.1 mm
Changed lines of the file:
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@@
-(kicad_pcb (version 4) (host pcbnew 4.0.7-e2-6376~58~ubuntu16.04.1)
+(kicad_pcb (version 20171130) (host pcbnew 5.0.2-bee76a0~70~ubuntu18.04.1)
   (general
-    (links 77)
-    (no_connects 0)
-    (area 49.924999 49.924999 100.075001 100.075001)
     (thickness 1.6)
     (drawings 11)
-    (tracks 41)
+    (tracks 44)
     (zones 0)
     (modules 23)
@@
   (page A4)
   (layers
-    (0 F.Cu signal)
+    (0 F.Cu signal hide)
     (31 B.Cu signal)
     (32 B.Adhes user hide)
@@
     (pad_drill 0.8)
     (pad_to_mask_clearance 0.2)
+    (solder_mask_min_width 0.25)
     (aux_axis_origin 0 0)
     (grid_origin 75 75)
@@
       (layerselection 0x010f0_80000001)
       (usegerberextensions false)
+      (usegerberattributes false)
+      (usegerberadvancedattributes false)
+      (creategerberjobfile false)
       (excludeedgelayer false)
       (linewidth 0.500000)
@@
       (hpglpennumber 1)
       (hpglpenspeed 20)
-      (hpglpendiameter 15)
-      (hpglpenoverlay 2)
+      (hpglpendiameter 15.000000)
       (psnegative false)
       (psa4output false)
@@
   )
   (module Fuse_Holders_and_Fuses:Fuseholder5x20_horiz_open_universal_Type-III (layer F.Cu)
-    (at 92.78 81.35 90)
+    (at 95.32 88.97 90)
     (descr "Fuseholder, 5x20, open, horizontal, Type-III, universal, inline, lateral,")
     (tags "Fuseholder 5x20 open horizontal Type-III universal inline lateral Sicherungshalter offen ")
@@
   )
   (module w_conn_pt-1,5:pt_1,5-2-3,5-h (layer F.Cu)
-    (at 75 54.045 180)
+    (at 95.955 61.665 90)
     (descr "2-way 3.5mm pitch terminal block, Phoenix PT series")
-    (fp_text reference J1 (at 0 5.08 180) (layer F.SilkS) hide
+    (fp_text reference J1 (at 0 5.08 90) (layer F.SilkS) hide
       (effects (font (size 1.5 1.5) (thickness 0.3)))
     )
-    (fp_text value Screw_Terminal_01x02 (at 0 -5 180) (layer F.SilkS) hide
+    (fp_text value Screw_Terminal_01x02 (at 0 -5 90) (layer F.SilkS) hide
       (effects (font (size 1.5 1.5) (thickness 0.3)))
     )
@@
     (fp_line (start 3.5 3.8) (end 3.5 -3.8) (layer F.SilkS) (width 0.381))
     (fp_line (start 3.5 -3.8) (end -3.5 -3.8) (layer F.SilkS) (width 0.381))
-    (pad 2 thru_hole circle (at -1.75 -0.7 180) (size 2.4 2.4) (drill 1.2) (layers *.Cu *.Mask F.SilkS)
+    (pad 2 thru_hole circle (at -1.75 -0.7 90) (size 2.4 2.4) (drill 1.2) (layers *.Cu *.Mask F.SilkS)
       (net 7 "Net-(F1-Pad2)"))
-    (pad 1 thru_hole rect (at 1.75 -0.7 180) (size 2.4 2.4) (drill 1.2) (layers *.Cu *.Mask F.SilkS)
+    (pad 1 thru_hole rect (at 1.75 -0.7 90) (size 2.4 2.4) (drill 1.2) (layers *.Cu *.Mask F.SilkS)
       (net 10 -V))
     (model Terminal_Blocks.3dshapes/Pheonix_MKDS1.5-2pol.wrl
@@
     (descr "TO-92 leads molded, narrow, drill 0.6mm (see NXP sot054_po.pdf)")
     (tags "to-92 sc-43 sc-43a sot54 PA33 transistor")
-    (fp_text reference Q1 (at -2.54 0 450) (layer F.SilkS)
+    (fp_text reference Q1 (at -2.54 0 90) (layer F.SilkS)
       (effects (font (size 1 1) (thickness 0.15)))
     )
@@
       (net 10 -V))
     (model ${KISYS3DMOD}/TO_SOT_Packages_THT.3dshapes/TO-92_Molded_Narrow.wrl
-      (at (xyz 0.05 0 0))
+      (offset (xyz 1.269999980926514 0 0))
       (scale (xyz 1 1 1))
       (rotate (xyz 0 0 -90))
@@
       (net 9 GND))
     (model TO_SOT_Packages_THT.3dshapes/TO-220_Vertical.wrl
-      (at (xyz 0.1 0 0))
+      (offset (xyz 2.539999961853027 0 0))
       (scale (xyz 0.4 0.4 0.4))
       (rotate (xyz 0 0 0))
@@
       (net 9 GND))
     (model TO_SOT_Packages_THT.3dshapes/TO-220_Vertical.wrl
-      (at (xyz 0.1 0 0))
+      (offset (xyz 2.539999961853027 0 0))
       (scale (xyz 0.4 0.4 0.4))
       (rotate (xyz 0 0 0))
@@
   (segment (start 59.76 63.57) (end 63.57 63.57) (width 0.75) (layer B.Cu) (net 1))
   (segment (start 71.19 63.57) (end 71.19 68.65) (width 0.75) (layer B.Cu) (net 2))
-  (segment (start 90.24 63.49) (end 92.78 60.95) (width 1.5) (layer B.Cu) (net 7))
-  (segment (start 95.32 63.49) (end 92.78 60.95) (width 1.5) (layer B.Cu) (net 7))
-  (segment (start 92.78 66.03) (end 95.32 63.49) (width 1.5) (layer B.Cu) (net 7))
-  (segment (start 90.24 63.49) (end 92.78 66.03) (width 1.5) (layer B.Cu) (net 7))
-  (segment (start 76.75 54.745) (end 76.97 54.745) (width 1.5) (layer B.Cu) (net 7))
-  (segment (start 86.51 59.76) (end 90.24 63.49) (width 1.5) (layer B.Cu) (net 7))
-  (segment (start 81.985 59.76) (end 86.51 59.76) (width 1.5) (layer B.Cu) (net 7))
-  (segment (start 76.97 54.745) (end 81.985 59.76) (width 1.5) (layer B.Cu) (net 7))
-  (segment (start 92.78 81.35) (end 90.24 78.81) (width 1.5) (layer B.Cu) (net 8))
-  (segment (start 92.78 81.35) (end 95.32 78.81) (width 1.5) (layer B.Cu) (net 8))
-  (segment (start 92.78 76.27) (end 95.32 78.81) (width 1.5) (layer B.Cu) (net 8))
-  (segment (start 90.24 78.81) (end 92.78 76.27) (width 1.5) (layer B.Cu) (net 8))
+  (segment (start 95.32 68.57) (end 95.32 63.48) (width 1.5) (layer F.Cu) (net 7))
+  (segment (start 95.32 63.48) (end 95.255 63.415) (width 1.5) (layer F.Cu) (net 7))
+  (segment (start 95.32 63.48) (end 95.255 63.415) (width 1.5) (layer B.Cu) (net 7))
+  (segment (start 95.32 63.48) (end 95.255 63.415) (width 1.5) (layer B.Cu) (net 7))
+  (segment (start 95.32 73.65) (end 92.78 71.11) (width 1.5) (layer B.Cu) (net 7))
+  (segment (start 92.78 71.11) (end 95.32 68.57) (width 1.5) (layer B.Cu) (net 7))
+  (segment (start 97.86 71.11) (end 95.32 68.57) (width 1.5) (layer B.Cu) (net 7))
+  (segment (start 95.32 73.65) (end 97.86 71.11) (width 1.5) (layer B.Cu) (net 7))
+  (segment (start 95.255 63.415) (end 95.255 63.635) (width 1.5) (layer B.Cu) (net 7) (status 30))
+  (segment (start 95.32 88.97) (end 92.78 86.43) (width 1.5) (layer B.Cu) (net 8))
+  (segment (start 97.86 86.43) (end 95.32 88.97) (width 1.5) (layer B.Cu) (net 8))
+  (segment (start 95.32 83.89) (end 97.86 86.43) (width 1.5) (layer B.Cu) (net 8))
+  (segment (start 92.78 86.43) (end 95.32 83.89) (width 1.5) (layer B.Cu) (net 8))
   (segment (start 78.175 60.395) (end 78.175 60.395) (width 1.5) (layer F.Cu) (net 8) (status 30))
   (segment (start 71.19 73.73) (end 70.174 73.73) (width 0.75) (layer B.Cu) (net 9) (status 30))
   (segment (start 71.19 73.73) (end 70.555 73.73) (width 0.75) (layer F.Cu) (net 9) (status 30))
+  (segment (start 95.255 59.915) (end 81.505 59.915) (width 1.5) (layer B.Cu) (net 10))
+  (segment (start 63.57 55.95) (end 63.57 53.41) (width 1.5) (layer B.Cu) (net 10))
+  (segment (start 65.475 57.855) (end 63.57 55.95) (width 1.5) (layer B.Cu) (net 10))
+  (segment (start 79.445 57.855) (end 65.475 57.855) (width 1.5) (layer B.Cu) (net 10))
+  (segment (start 81.505 59.915) (end 79.445 57.855) (width 1.5) (layer B.Cu) (net 10))
   (segment (start 72.46 86.35) (end 72.38 86.43) (width 1.5) (layer F.Cu) (net 10) (status 30))
   (segment (start 57.22 76.27) (end 57.22 73.095) (width 0.75) (layer B.Cu) (net 11))
@@
   (segment (start 57.22 76.27) (end 57.22 75.635) (width 0.75) (layer B.Cu) (net 11) (status 30))
   (segment (start 78.81 73.73) (end 78.81 71.19) (width 0.75) (layer B.Cu) (net 12))
-  (segment (start 83.89 53.41) (end 78.81 53.41) (width 0.75) (layer B.Cu) (net 13))
-  (segment (start 70.555 53.537) (end 70.555 60.395) (width 0.75) (layer B.Cu) (net 13))
-  (segment (start 71.444 52.648) (end 70.555 53.537) (width 0.75) (layer B.Cu) (net 13))
-  (segment (start 78.048 52.648) (end 71.444 52.648) (width 0.75) (layer B.Cu) (net 13))
-  (segment (start 78.81 53.41) (end 78.048 52.648) (width 0.75) (layer B.Cu) (net 13))
+  (segment (start 70.555 60.395) (end 77.54 53.41) (width 0.75) (layer F.Cu) (net 13))
+  (segment (start 77.54 53.41) (end 83.89 53.41) (width 0.75) (layer F.Cu) (net 13))
   (segment (start 70.555 60.395) (end 70.555 60.395) (width 0.75) (layer B.Cu) (net 13) (status 30))
   (segment (start 70.555 60.395) (end 64.205 60.395) (width 0.75) (layer B.Cu) (net 13) (status 10))

Commit message: tunk
Other:
- net class Default removed
