File: dual-pwr/dual-pwr.sch (KiCad schematic (older format))
At the start: 24 parts, among them J1 Screw_Terminal_01x02, J2 Screw_Terminal_01x03, J3 Conn_01x01, J4 Conn_01x01, J5 Conn_01x01, J6 Conn_01x01, Q1 2N3904, Q2 TIP122, Q3 TIP127, U1 NE5532

Commit message: dual-pwr
Parts:
- C1, C2: value 10u 35V -> 1000u 25V
- C3, C4: value 100n -> 1u 50V
- D1, D2: value D -> 2N4007
- D3: value D -> 1N5822
- R3: value 10k -> 470k
- R4: value 4k7 -> 2k2
Connections:
- net -V: now reaches C2.2, C4.2, D2.2 (A), D3.2 (A), J1.1 (Pin_1), J2.3 (Pin_3), Q1.1 (E), Q3.2 (C), R2.2, R6.2, U1.4 (V-)
- net +V: now reaches C1.1, C3.1, D1.1 (K), D3.1 (K), F1.1, J2.1 (Pin_1), Q2.2 (C), R1.1, R4.1, R5.1, U1.8 (V+)
- net GND: now reaches C1.2, C2.1, C3.2, C4.1, D1.2 (A), D2.1 (K), J2.2 (Pin_2), Q2.3 (E), Q3.3 (E), R5.2, R6.1, U1.5 (+)
Changed lines of the file:
@@
 P 5000 3850
 F 0 "R3" V 5080 3850 50  0000 C CNN
-F 1 "10k" V 5000 3850 50  0000 C CNN
+F 1 "470k" V 5000 3850 50  0000 C CNN
 F 2 "Resistors_ThroughHole:R_Axial_DIN0207_L6.3mm_D2.5mm_P7.62mm_Horizontal" V 4930 3850 50  0001 C CNN
 F 3 "" H 5000 3850 50  0001 C CNN
@@
 P 5500 2850
 F 0 "R4" V 5580 2850 50  0000 C CNN
-F 1 "4k7" V 5500 2850 50  0000 C CNN
+F 1 "2k2" V 5500 2850 50  0000 C CNN
 F 2 "Resistors_ThroughHole:R_Axial_DIN0207_L6.3mm_D2.5mm_P7.62mm_Horizontal" V 5430 2850 50  0001 C CNN
 F 3 "" H 5500 2850 50  0001 C CNN
@@
 P 7800 3100
 F 0 "C1" H 7825 3200 50  0000 L CNN
-F 1 "10u 35V" H 7825 3000 50  0000 L CNN
+F 1 "1000u 25V" H 7825 3000 50  0000 L CNN
 F 2 "Capacitors_ThroughHole:CP_Radial_D10.0mm_P3.50mm" H 7838 2950 50  0001 C CNN
 F 3 "" H 7800 3100 50  0001 C CNN
@@
 P 7800 4300
 F 0 "C2" H 7825 4400 50  0000 L CNN
-F 1 "10u 35V" H 7825 4200 50  0000 L CNN
+F 1 "1000u 25V" H 7825 4200 50  0000 L CNN
 F 2 "Capacitors_ThroughHole:CP_Radial_D10.0mm_P3.50mm" H 7838 4150 50  0001 C CNN
 F 3 "" H 7800 4300 50  0001 C CNN
@@
 P 8300 3100
 F 0 "C3" H 8325 3200 50  0000 L CNN
-F 1 "100n" H 8325 3000 50  0000 L CNN
+F 1 "1u 50V" H 8325 3000 50  0000 L CNN
 F 2 "Capacitors_ThroughHole:C_Rect_L7.0mm_W4.5mm_P5.00mm" H 8338 2950 50  0001 C CNN
 F 3 "" H 8300 3100 50  0001 C CNN
@@
 P 8300 4300
 F 0 "C4" H 8325 4400 50  0000 L CNN
-F 1 "100n" H 8325 4200 50  0000 L CNN
+F 1 "1u 50V" H 8325 4200 50  0000 L CNN
 F 2 "Capacitors_ThroughHole:C_Rect_L7.0mm_W4.5mm_P5.00mm" H 8338 4150 50  0001 C CNN
 F 3 "" H 8300 4300 50  0001 C CNN
@@
 	5500 3000 5500 4500
 Wire Wire Line
-	6000 3600 8750 3600
+	5850 3600 8750 3600
 Wire Wire Line
 	7800 2500 7800 2950
@@
 P 3100 3600
 F 0 "D3" H 3100 3700 50  0000 C CNN
-F 1 "D" H 3100 3500 50  0000 C CNN
+F 1 "1N5822" H 3100 3500 50  0000 C CNN
 F 2 "Diodes_ThroughHole:D_DO-27_P15.24mm_Horizontal" H 3100 3600 50  0001 C CNN
 F 3 "" H 3100 3600 50  0001 C CNN
@@
 	2350 2500 8600 2500
 Wire Wire Line
-	3100 3750 3100 5050
+	3100 3750 3100 5350
 Connection ~ 3100 5050
 $Comp
@@
 	1650 2500 2050 2500
 Wire Wire Line
-	3100 3450 3100 2500
+	3100 2250 3100 3450
 Connection ~ 3100 2500
 $Comp
@@
 P 6850 3100
 F 0 "D1" H 6850 3200 50  0000 C CNN
-F 1 "D" H 6850 3000 50  0000 C CNN
+F 1 "2N4007" H 6850 3000 50  0000 C CNN
 F 2 "Diodes_ThroughHole:D_DO-41_SOD81_P10.16mm_Horizontal" H 6850 3100 50  0001 C CNN
 F 3 "" H 6850 3100 50  0001 C CNN
@@
 P 6850 4300
 F 0 "D2" H 6850 4400 50  0000 C CNN
-F 1 "D" H 6850 4200 50  0000 C CNN
+F 1 "2N4007" H 6850 4200 50  0000 C CNN
 F 2 "Diodes_ThroughHole:D_DO-41_SOD81_P10.16mm_Horizontal" H 6850 4300 50  0001 C CNN
 F 3 "" H 6850 4300 50  0001 C CNN
@@
 	7250 4450 7250 5050
 Connection ~ 7250 5050
+Text GLabel 3100 2250 1    60   Input ~ 0
++V
+Text GLabel 3100 5350 3    60   Input ~ 0
+-V
+Text GLabel 5850 3600 0    60   Input ~ 0
+GND
 $EndSCHEMATC

Commit message: dual-pwr
Parts:
- removed R5, R6: 10k, Resistors_ThroughHole:R_Axial_DIN0207_L6.3mm_D2.5mm_P7.62mm_Horizontal, symbol R
- added RV1: 2k, Potentiometers:Potentiometer_Trimmer_Vishay_T73XW_Vertical, symbol POT
- C1, C2: footprint Capacitors_ThroughHole:CP_Radial_D10.0mm_P3.50mm -> Capacitors_ThroughHole:CP_Radial_D10.0mm_P5.00mm
- C3, C4: footprint Capacitors_ThroughHole:C_Rect_L7.0mm_W4.5mm_P5.00mm -> Capacitors_ThroughHole:C_Disc_D5.0mm_W2.5mm_P5.00mm
- R2: value 10k -> 9k1
Connections:
- net +V: now also U1.8 (V+); no longer U1.8 (V+)
- net -V: now also U1.4 (V-), RV1.2, RV1.3; no longer R2.2, U1.4 (V-)
- net GND: now also U1.3 (+); no longer U1.5 (+)
- net Vref: now reaches R1.2, R2.1
- net Vref: now also U1.2 (-), U1.5 (+); no longer U1.3 (+), U1.6 (-)
- net at U1.7: now also U1.6 (-); no longer R3.1
- net at U1.1: now also R3.1; no longer U1.2 (-)
- net VBase: now reaches Q1.3 (C), Q2.1 (B), Q3.1 (B), R4.2
- new net: R2.2, RV1.1
Other:
- moved on the sheet: U1A, U1B
Changed lines of the file:
@@
 EESchema Schematic File Version 2
-LIBS:dual-pwr-rescue
 LIBS:power
 LIBS:device
@@
 L NE5532 U1
 U 2 1 5AA67495
+P 4300 5800
+F 0 "U1" H 4300 6000 50  0000 L CNN
+F 1 "NE5532" H 4300 5600 50  0000 L CNN
+F 2 "Housings_DIP:DIP-8_W7.62mm_Socket" H 4300 5800 50  0001 C CNN
+F 3 "" H 4300 5800 50  0001 C CNN
+	2    4300 5800
+	1    0    0    -1
+$EndComp
+$Comp
+L NE5532 U1
+U 1 1 5AA6759E
 P 4500 3500
 F 0 "U1" H 4500 3700 50  0000 L CNN
@@
 F 2 "Housings_DIP:DIP-8_W7.62mm_Socket" H 4500 3500 50  0001 C CNN
 F 3 "" H 4500 3500 50  0001 C CNN
-	2    4500 3500
-	1    0    0    -1
-$EndComp
-$Comp
-L NE5532 U1
-U 1 1 5AA6759E
-P 4300 5800
-F 0 "U1" H 4300 6000 50  0000 L CNN
-F 1 "NE5532" H 4300 5600 50  0000 L CNN
-F 2 "Housings_DIP:DIP-8_W7.62mm_Socket" H 4300 5800 50  0001 C CNN
-F 3 "" H 4300 5800 50  0001 C CNN
-	1    4300 5800
+	1    4500 3500
 	1    0    0    -1
 $EndComp
@@
 P 3600 3850
 F 0 "R2" V 3680 3850 50  0000 C CNN
-F 1 "10k" V 3600 3850 50  0000 C CNN
+F 1 "9k1" V 3600 3850 50  0000 C CNN
 F 2 "Resistors_ThroughHole:R_Axial_DIN0207_L6.3mm_D2.5mm_P7.62mm_Horizontal" V 3530 3850 50  0001 C CNN
 F 3 "" H 3600 3850 50  0001 C CNN
@@
 F 0 "C1" H 7825 3200 50  0000 L CNN
 F 1 "1000u 25V" H 7825 3000 50  0000 L CNN
-F 2 "Capacitors_ThroughHole:CP_Radial_D10.0mm_P3.50mm" H 7838 2950 50  0001 C CNN
+F 2 "Capacitors_ThroughHole:CP_Radial_D10.0mm_P5.00mm" H 7838 2950 50  0001 C CNN
 F 3 "" H 7800 3100 50  0001 C CNN
 	1    7800 3100
@@
 F 0 "C2" H 7825 4400 50  0000 L CNN
 F 1 "1000u 25V" H 7825 4200 50  0000 L CNN
-F 2 "Capacitors_ThroughHole:CP_Radial_D10.0mm_P3.50mm" H 7838 4150 50  0001 C CNN
+F 2 "Capacitors_ThroughHole:CP_Radial_D10.0mm_P5.00mm" H 7838 4150 50  0001 C CNN
 F 3 "" H 7800 4300 50  0001 C CNN
 	1    7800 4300
@@
 F 0 "C3" H 8325 3200 50  0000 L CNN
 F 1 "1u 50V" H 8325 3000 50  0000 L CNN
-F 2 "Capacitors_ThroughHole:C_Rect_L7.0mm_W4.5mm_P5.00mm" H 8338 2950 50  0001 C CNN
+F 2 "Capacitors_ThroughHole:C_Disc_D5.0mm_W2.5mm_P5.00mm" H 8338 2950 50  0001 C CNN
 F 3 "" H 8300 3100 50  0001 C CNN
 	1    8300 3100
@@
 F 0 "C4" H 8325 4400 50  0000 L CNN
 F 1 "1u 50V" H 8325 4200 50  0000 L CNN
-F 2 "Capacitors_ThroughHole:C_Rect_L7.0mm_W4.5mm_P5.00mm" H 8338 4150 50  0001 C CNN
+F 2 "Capacitors_ThroughHole:C_Disc_D5.0mm_W2.5mm_P5.00mm" H 8338 4150 50  0001 C CNN
 F 3 "" H 8300 4300 50  0001 C CNN
 	1    8300 4300
@@
 Connection ~ 3600 2500
 Wire Wire Line
-	3600 4000 3600 5050
-Connection ~ 3600 5050
-Wire Wire Line
 	3600 3500 3600 3700
 Wire Wire Line
@@
 	4000 6250 4000 5900
 Wire Wire Line
-	4000 5700 4000 3600
+	4000 3400 4000 5700
 Connection ~ 4000 3600
 $Comp
@@
 Connection ~ 5500 4000
 Wire Wire Line
-	5700 3100 5500 3100
+	5300 3100 5700 3100
 Connection ~ 5500 3100
 Wire Wire Line
@@
 Connection ~ 6000 5050
 Connection ~ 6000 3600
-$Comp
-L R R5
-U 1 1 5AA7059C
-P 7250 3100
-F 0 "R5" V 7330 3100 50  0000 C CNN
-F 1 "10k" V 7250 3100 50  0000 C CNN
-F 2 "Resistors_ThroughHole:R_Axial_DIN0207_L6.3mm_D2.5mm_P7.62mm_Horizontal" V 7180 3100 50  0001 C CNN
-F 3 "" H 7250 3100 50  0001 C CNN
-	1    7250 3100
-	1    0    0    -1
-$EndComp
-$Comp
-L R R6
-U 1 1 5AA70627
-P 7250 4300
-F 0 "R6" V 7330 4300 50  0000 C CNN
-F 1 "10k" V 7250 4300 50  0000 C CNN
-F 2 "Resistors_ThroughHole:R_Axial_DIN0207_L6.3mm_D2.5mm_P7.62mm_Horizontal" V 7180 4300 50  0001 C CNN
-F 3 "" H 7250 4300 50  0001 C CNN
-	1    7250 4300
-	1    0    0    -1
-$EndComp
-Wire Wire Line
-	7250 2950 7250 2500
-Connection ~ 7250 2500
 Wire Wire Line
 	6850 2950 6850 2500
@@
 Connection ~ 6850 3600
 Wire Wire Line
-	7250 3250 7250 4150
-Connection ~ 7250 3600
-Wire Wire Line
 	6850 4450 6850 5050
 Connection ~ 6850 5050
-Wire Wire Line
-	7250 4450 7250 5050
-Connection ~ 7250 5050
 Text GLabel 3100 2250 1    60   Input ~ 0
 +V
@@
 Text GLabel 5850 3600 0    60   Input ~ 0
 GND
+$Comp
+L POT RV1
+U 1 1 5ACA1980
+P 3600 4400
+F 0 "RV1" V 3425 4400 50  0000 C CNN
+F 1 "2k" V 3500 4400 50  0000 C CNN
+F 2 "Potentiometers:Potentiometer_Trimmer_Vishay_T73XW_Vertical" H 3600 4400 50  0001 C CNN
+F 3 "" H 3600 4400 50  0001 C CNN
+	1    3600 4400
+	1    0    0    -1
+$EndComp
+Wire Wire Line
+	3600 4250 3600 4000
+Wire Wire Line
+	3600 4550 3600 5050
+Connection ~ 3600 5050
+Wire Wire Line
+	3750 4400 3750 4650
+Wire Wire Line
+	3750 4650 3600 4650
+Connection ~ 3600 4650
+Text GLabel 5300 3100 0    60   Input ~ 0
+VBase
+Text GLabel 4000 3400 1    60   Input ~ 0
+Vref
 $EndSCHEMATC
