File: blink-timer/blink-timer.kicad_pcb (KiCad board)
At the start: 2 copper layers, 44 x 21 mm, 14 parts, among them J1 Conn_01x04_Socket, Q1 IRF4905, U1 LM393

Commit message: tunk
Parts:
- moved J1 12.7 mm to (117.6, 118.0), turned to 90 degrees
- moved R6 9.24 mm to (131.5, 104.0)
- moved R5 9.23 mm to (127.0, 104.0)
- moved D3 9.14 mm to (128.5, 118.0)
- moved D2 4.71 mm to (127.5, 111.0), turned to 0 degrees
- moved D1 4.26 mm to (127.5, 114.0), turned to 180 degrees
- moved R2 3.45 mm to (132.7, 109.0)
- moved R3 3.20 mm to (132.7, 113.0), turned to -90 degrees
- moved C1 3.03 mm to (139.0, 105.0)
- moved R1 2.96 mm to (138.5, 102.5)
- moved C2 2.59 mm to (139.0, 108.0)
- moved U1 2.02 mm to (138.5, 113.0)
Routing:
- net Net-(D1-A): track 15.8 -> 25.7 mm, vias 2 -> 0
- net Net-(J1-Pin_2): track 25.2 -> 20.0 mm
- net GND: track 13.4 -> 9.03 mm, vias 4 -> 5
- net +12V: track 27.8 -> 25.6 mm
- net IN: track 8.64 -> 10.1 mm, vias 1 -> 0
- net VCC: track 3.50 -> 2.39 mm

Commit message: tunk
Routing:
- net VCC: track 2.39 -> 8.41 mm, vias 0 -> 2
- net Net-(J1-Pin_2): track 20.0 -> 19.0 mm
Changed lines of the file:
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@@
 			(plot_on_all_layers_selection 0x0000000_00000000)
 			(disableapertmacros no)
-			(usegerberextensions no)
-			(usegerberattributes yes)
-			(usegerberadvancedattributes yes)
-			(creategerberjobfile yes)
+			(usegerberextensions yes)
+			(usegerberattributes no)
+			(usegerberadvancedattributes no)
+			(creategerberjobfile no)
 			(dashed_line_dash_ratio 12.000000)
 			(dashed_line_gap_ratio 3.000000)
@@
 			(psa4output no)
 			(plotreference yes)
-			(plotvalue yes)
+			(plotvalue no)
 			(plotfptext yes)
 			(plotinvisibletext no)
 			(sketchpadsonfab no)
-			(subtractmaskfromsilk no)
+			(subtractmaskfromsilk yes)
 			(outputformat 1)
 			(mirror no)
-			(drillshape 1)
+			(drillshape 0)
 			(scaleselection 1)
-			(outputdirectory "")
+			(outputdirectory "plot")
 		)
 	)
@@
 		(tags "resistor handsolder")
 		(property "Reference" "R2"
-			(at 0 -1.5 90)
+			(at -0.034 1.651 90)
 			(layer "F.SilkS")
 			(effects
@@
 		(tags "resistor handsolder")
 		(property "Reference" "R5"
-			(at 1 -1.5 0)
+			(at -0.508 1.664 0)
 			(layer "F.SilkS")
 			(effects
@@
 		(tags "resistor handsolder")
 		(property "Reference" "R6"
-			(at -1 -1.65 0)
+			(at 1.088 1.664 0)
 			(layer "F.SilkS")
 			(effects
@@
 		(tags "SOIC SO")
 		(property "Reference" "U1"
-			(at 0 3.5 0)
+			(at 0 0 0)
 			(layer "F.SilkS")
 			(effects
@@
 		(tags "Diode Mini-MELF (SOD-80)")
 		(property "Reference" "D2"
-			(at 0 0 360)
+			(at 0 0 0)
 			(layer "F.SilkS")
 			(effects
@@
 		)
 		(property "Value" "1N4148"
-			(at 0 2 360)
+			(at 0 2 0)
 			(layer "F.Fab")
 			(effects
@@
 		)
 		(fp_text user "${REFERENCE}"
-			(at 0 -2 360)
+			(at 0 -2 0)
 			(layer "F.Fab")
 			(effects
@@
 		(tags "resistor handsolder")
 		(property "Reference" "R3"
-			(at 0 -1.65 90)
+			(at -0.478 1.651 90)
 			(layer "F.SilkS")
 			(effects
@@
 		(tags "Diode SMA (DO-214AC)")
 		(property "Reference" "D3"
-			(at -4.5 -1.5 180)
+			(at -4.342 -0.11 180)
 			(layer "F.SilkS")
 			(effects
@@
 		(tags "Altech AK100 serie connector")
 		(property "Reference" "J1"
-			(at -1.0765 -3.7425 270)
+			(at -1.0765 -3.7425 -90)
 			(layer "F.SilkS")
 			(effects
@@
 		)
 		(property "Value" "Conn_01x04_Socket"
-			(at 7.5 5.25 270)
+			(at 7.5 5.25 -90)
 			(layer "F.Fab")
 			(effects
@@
 		)
 		(fp_text user "${REFERENCE}"
-			(at 7.5 -0.5 270)
+			(at 7.5 -0.5 -90)
 			(layer "F.Fab")
 			(effects
@@
 	)
 	(gr_text "DRL delay\nsjm 2024/05"
-		(at 123.19 114.3 0)
+		(at 141.732 105.918 0)
 		(layer "B.SilkS")
 		(effects
@@
 	)
 	(gr_text "OUT"
-		(at 122.5 128 270)
+		(at 122.5 111.252 -90)
 		(layer "F.SilkS")
 		(effects
@@
 	)
 	(gr_text "IN"
-		(at 127 126 270)
+		(at 122.428 106.68 -90)
 		(layer "F.SilkS")
 		(effects
@@
 		)
 	)
-	(gr_text "sjm\n2024/05"
-		(at 106.5 131.5 0)
+	(gr_text "sjm 2024/05"
+		(at 124.968 102.108 0)
 		(layer "F.SilkS")
 		(effects
@@
 	)
 	(gr_text "DRL\ndelay"
-		(at 148.5 97.5 0)
+		(at 137.16 119.38 0)
 		(layer "F.SilkS")
 		(effects
@@
 	)
 	(gr_text "GND"
-		(at 132 128 -90)
+		(at 122.428 101.092 -90)
 		(layer "F.SilkS")
 		(effects
@@
 	)
 	(gr_text "+12V"
-		(at 118 126.5 270)
+		(at 122.428 115.316 270)
 		(layer "F.SilkS")
 		(effects
@@
 	)
 	(segment
-		(start 132.715 114)
-		(end 132.715 114.3)
-		(width 0.508)
-		(layer "F.Cu")
-		(net 3)
-	)
-	(segment
 		(start 138.38 108)
 		(end 137.4375 108)
@@
 	)
 	(segment
-		(start 137.5 104.9375)
-		(end 137.4375 105)
-		(width 0.508)
-		(layer "F.Cu")
-		(net 5)
-	)
-	(segment
 		(start 140.975 113.635)
 		(end 139.67 113.635)
@@
 	)
 	(segment
-		(start 132.715 112)
-		(end 132.955 112)
-		(width 0.508)
-		(layer "F.Cu")
-		(net 6)
-	)
-	(segment
 		(start 132.715 110)
 		(end 132.715 112)
@@
 	)
 	(segment
+		(start 129.286 106.299)
+		(end 129.286 105.156)
+		(width 0.508)
+		(layer "F.Cu")
+		(net 8)
+	)
+	(segment
 		(start 132.715 108)
 		(end 130.987 108)
@@
 	)
 	(segment
-		(start 130.987 108)
-		(end 130.937 107.95)
+		(start 129.286 106.299)
+		(end 130.987 108)
 		(width 0.508)
 		(layer "F.Cu")
 		(net 8)
 	)
+	(via
+		(at 129.286 105.156)
+		(size 0.6)
+		(drill 0.3)
+		(layers "F.Cu" "B.Cu")
+		(net 8)
+	)
+	(via
+		(at 129.286 102.616)
+		(size 0.6)
+		(drill 0.3)
+		(layers "F.Cu" "B.Cu")
+		(net 8)
+	)
 	(segment
-		(start 117.5675 113)
-		(end 115 113)
+		(start 129.286 105.156)
+		(end 129.286 102.616)
 		(width 1.016)
-		(layer "F.Cu")
-		(net 9)
+		(layer "B.Cu")
+		(net 8)
 	)
 	(segment
-		(start 109.85 107.85)
-		(end 108.82 107.85)
+		(start 117.5675 113)
+		(end 115 113)
 		(width 1.016)
 		(layer "F.Cu")
